File: io.kicad_sch (KiCad schematic)
At the start: 8 parts

Commit message: Remapped GPIOs for clean routing
This updates the GPIO table so that the traces and vias are far cleaner. Slight repositioning of some pins to account for that. Rebuilt all gerbers and necessary stuff.
Connections:
- net GPIO35 renamed GPIO11
- net GPIO39 renamed GPIO12
- net GPIO40 renamed GPIO13
- net GPIO41 renamed GPIO14
- net GPIO42 renamed GPIO9
- net GPIO45 renamed GPIO10
Changed lines of the file:
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@@
+		)
+	)
+	(hierarchical_label "GPIO11"
+		(shape bidirectional)
+		(at 38.1 44.45 0)
+		(fields_autoplaced yes)
+		(effects
+			(font
+				(size 1.27 1.27)
+			)
+			(justify left)
+		)
+		(property "GPIO11" ""
+			(at 38.1 45.72 0)
+			(effects
+				(font
+					(size 1.27 1.27)
+					(italic yes)
+				)
+				(justify left)
+			)
 		)
 	)
@@
 		)
 	)
-	(hierarchical_label "GPIO41"
+	(hierarchical_label "GPIO14"
 		(shape bidirectional)
 		(at 92.71 44.45 0)
@@
 			(justify left)
 		)
-		(property "GPIO41" ""
+		(property "GPIO14" ""
 			(at 92.71 45.72 0)
 			(effects
@@
 		)
 	)
-	(hierarchical_label "GPIO45"
+	(hierarchical_label "GPIO10"
 		(shape bidirectional)
 		(at 129.54 44.45 0)
-		(fields_autoplaced yes)
 		(effects
 			(font
@@
 			(justify left)
 		)
-		(property "GPIO45" ""
-			(at 129.54 45.72 0)
-			(effects
-				(font
-					(size 1.27 1.27)
-					(italic yes)
-				)
-				(justify left)
-			)
-		)
 	)
-	(hierarchical_label "GPIO42"
+	(hierarchical_label "GPIO9"
 		(shape bidirectional)
 		(at 111.76 44.45 0)
@@
 			(justify left)
 		)
-		(property "GPIO42" ""
+		(property "GPIO9" ""
 			(at 111.76 45.72 0)
 			(effects
@@
 		)
 	)
-	(hierarchical_label "GPIO39"
+	(hierarchical_label "GPIO12"
 		(shape bidirectional)
 		(at 55.88 44.45 0)
@@
 			(justify left)
 		)
-		(property "GPIO39" ""
+		(property "GPIO10" ""
 			(at 55.88 45.72 0)
 			(effects
@@
 		)
 	)
-	(hierarchical_label "GPIO35"
-		(shape bidirectional)
-		(at 38.1 44.45 0)
-		(fields_autoplaced yes)
-		(effects
-			(font
-				(size 1.27 1.27)
-			)
-			(justify left)
-		)
-		(property "GPIO35" ""
-			(at 38.1 45.72 0)
-			(effects
-				(font
-					(size 1.27 1.27)
-					(italic yes)
-				)
-				(justify left)
-			)
-		)
-	)
-	(hierarchical_label "GPIO40"
+	(hierarchical_label "GPIO13"
 		(shape bidirectional)
 		(at 73.66 44.45 0)
@@
 			(justify left)
 		)
-		(property "GPIO40" ""
+		(property "GPIO11" ""
 			(at 73.66 45.72 0)
 			(effects

Commit message: Updated to v1.1 to fix issues
Parts:
- removed J_Digital5: D5, Connector_PinHeader_2.54mm:PinHeader_1x03_P2.54mm_Vertical, symbol Connector:Conn_01x03_Pin
- removed J_Digital6: D6, Connector_PinHeader_2.54mm:PinHeader_1x03_P2.54mm_Vertical, symbol Connector:Conn_01x03_Pin
Connections:
- net GPIO11 renamed GPIO39
- net GPIO12 renamed GPIO40
- net GPIO13 renamed GPIO41
- net GPIO14 renamed GPIO42
