File: rc_control.kicad_sch (KiCad schematic)
At the start: 3 parts

Commit message: Remapped GPIOs for clean routing
This updates the GPIO table so that the traces and vias are far cleaner. Slight repositioning of some pins to account for that. Rebuilt all gerbers and necessary stuff.
Connections:
- net GPIO39 renamed GPIO12
- net GPIO48 renamed GPIO13
Changed lines of the file:
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@@
 		)
 	)
-	(hierarchical_label "GPIO39"
+	(hierarchical_label "GPIO12"
 		(shape bidirectional)
 		(at 82.55 55.88 0)
-		(fields_autoplaced yes)
 		(effects
 			(font
@@
 			(justify left)
 		)
-		(property "GPIO39" ""
-			(at 82.55 57.15 0)
-			(effects
-				(font
-					(size 1.27 1.27)
-					(italic yes)
-				)
-				(justify left)
-			)
-		)
 	)
-	(hierarchical_label "GPIO48"
+	(hierarchical_label "GPIO13"
 		(shape bidirectional)
 		(at 82.55 58.42 0)
-		(fields_autoplaced yes)
 		(effects
 			(font
@@
 			(justify left)
 		)
-		(property "GPIO48" ""
-			(at 82.55 59.69 0)
-			(effects
-				(font
-					(size 1.27 1.27)
-					(italic yes)
-				)
-				(justify left)
-			)
-		)
 	)

Commit message: Updated to v1.1 to fix issues
Parts:
- removed J_RCSEL1: RCSEL, Connector_PinHeader_2.54mm:PinHeader_1x02_P2.54mm_Vertical, symbol Connector:Conn_01x02_Pin
- removed J_SEL2: RCSEL2, Connector_PinHeader_2.54mm:PinHeader_1x02_P2.54mm_Vertical, symbol Connector:Conn_01x02_Pin
Other:
- note removed: "mutually exclusive with SW-UART"
- note removed: "shared with Digital 2 - mutually exclusive"
Changed lines of the file:
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@@
 	(generator_version "9.0")
 	(paper "A4")
-	(text "mutually exclusive with SW-UART"
-		(exclude_from_sim no)
-		(at 98.806 73.66 0)
-		(effects
-			(font
-				(size 1.27 1.27)
-			)
-		)
-	)
-	(text "shared with Digital 2 - mutually exclusive"
-		(exclude_from_sim no)
-		(at 105.664 51.054 0)
-		(effects
-			(font
-				(size 1.27 1.27)
-			)
-		)
-	)
-	(hierarchical_label "GPIO38"
-		(shape bidirectional)
-		(at 82.55 81.28 0)
-		(fields_autoplaced yes)
-		(effects
-			(font
-				(size 1.27 1.27)
-			)
-			(justify left)
-		)
-		(property "GPIO38" ""
-			(at 82.55 82.55 0)
-			(effects
-				(font
-					(size 1.27 1.27)
-					(italic yes)
-				)
-				(justify left)
-			)
-		)
-	)
 	(hierarchical_label "GPIO47"
 		(shape bidirectional)
@@
 				(justify left)
 			)
-		)
-	)
-	(hierarchical_label "GPIO21"
-		(shape bidirectional)
-		(at 82.55 78.74 0)
-		(fields_autoplaced yes)
-		(effects
-			(font
-				(size 1.27 1.27)
-			)
-			(justify left)
-		)
-		(property "GPIO21" ""
-			(at 82.55 80.01 0)
-			(effects
-				(font
-					(size 1.27 1.27)
-					(italic yes)
-				)
-				(justify left)
-			)
-		)
-	)
-	(hierarchical_label "GPIO12"
-		(shape bidirectional)
-		(at 82.55 55.88 0)
-		(effects
-			(font
-				(size 1.27 1.27)
-			)
-			(justify left)
-		)
-	)
-	(hierarchical_label "GPIO13"
-		(shape bidirectional)
-		(at 82.55 58.42 0)
-		(effects
-			(font
-				(size 1.27 1.27)
-			)
-			(justify left)
 		)
 	)
@@
 	)
 	(symbol
-		(lib_id "Connector:Conn_01x02_Pin")
-		(at 77.47 78.74 0)
-		(unit 1)
-		(exclude_from_sim no)
-		(in_bom yes)
-		(on_board yes)
-		(dnp no)
-		(fields_autoplaced yes)
-		(property "Reference" "J_SEL2"
-			(at 78.105 73.66 0)
-			(effects
-				(font
-					(size 1.27 1.27)
-				)
-			)
-		)
-		(property "Value" "RCSEL2"
-			(at 78.105 76.2 0)
-			(effects
-				(font
-					(size 1.27 1.27)
-				)
-			)
-		)
-		(property "Footprint" "Connector_PinHeader_2.54mm:PinHeader_1x02_P2.54mm_Vertical"
-			(at 77.47 78.74 0)
-			(effects
-				(font
-					(size 1.27 1.27)
-				)
-				(hide yes)
-			)
-		)
-		(property "Datasheet" "~"
-			(at 77.47 78.74 0)
-			(effects
-				(font
-					(size 1.27 1.27)
-				)
-				(hide yes)
-			)
-		)
-		(property "Description" "Generic connector, single row, 01x02, script generated"
-			(at 77.47 78.74 0)
-			(effects
-				(font
-					(size 1.27 1.27)
-				)
-				(hide yes)
-			)
-		)
-		(pin "2"
-		)
-		(pin "1"
-		)
-		(instances
-			(project "AmidalaShield"
-				(path "/6d8d0000-f03d-4277-95db-0f566c3960c4/e4484725-300e-4e40-a7d6-a015a6cb4529"
-					(reference "J_SEL2")
-					(unit 1)
-				)
-			)
-		)
-	)
-	(symbol
 		(lib_id "power:GND")
 		(at 57.15 54.61 90)
@@
 					(unit 1)
 				)
-			)
-		)
-	)
-	(symbol
-		(lib_id "Connector:Conn_01x02_Pin")
-		(at 77.47 55.88 0)
-		(unit 1)
-		(exclude_from_sim no)
-		(in_bom yes)
-		(on_board yes)
-		(dnp no)
-		(fields_autoplaced yes)
-		(property "Reference" "J_RCSEL1"
-			(at 78.105 50.8 0)
-			(effects
-				(font
-					(size 1.27 1.27)
-				)
-			)
-		)
-		(property "Value" "RCSEL"
-			(at 78.105 53.34 0)
-			(effects
-				(font
-					(size 1.27 1.27)
-				)
-			)
-		)
-		(property "Footprint" "Connector_PinHeader_2.54mm:PinHeader_1x02_P2.54mm_Vertical"
-			(at 77.47 55.88 0)
-			(effects
-				(font
-					(size 1.27 1.27)
-				)
-				(hide yes)
-			)
-		)
-		(property "Datasheet" "~"
-			(at 77.47 55.88 0)
-			(effects
-				(font
-					(size 1.27 1.27)
-				)
-				(hide yes)
-			)
-		)
-		(property "Description" "Generic connector, single row, 01x02, script generated"
-			(at 77.47 55.88 0)
-			(effects
-				(font
-					(size 1.27 1.27)
-				)
-				(hide yes)
-			)
-		)
-		(pin "2"
-		)
-		(pin "1"
-		)
-		(instances
-			(project "AmidalaShield"
-				(path "/6d8d0000-f03d-4277-95db-0f566c3960c4/e4484725-300e-4e40-a7d6-a015a6cb4529"
-					(reference "J_RCSEL1")
-					(unit 1)
-				)
